Commit message: Tuned URDF parameters

File: src/magician-master/urdf/demo.urdf (robot description, URDF)
Before this commit: robot magician, 6 links, 5 joints
Joints:
- joint joint_2: origin xyz=-0.01175 0 0.114 rpy=1.570796325 0 -1.570796325 -> xyz=-0.01175 0 0.114 rpy=1.570796325 -0.2 0
- joint joint_5: origin xyz=0.02699 0.13228 -0.01175 rpy=0 3.14159265 0 -> xyz=0.02699 0.13228 -0.01175 rpy=0 3.14159265 0.4

Commit message: Added joystick control under simulation, fixed joint linkage offset problem

File: src/magician-master/urdf/demo.urdf (robot description, URDF)
Before this commit: robot magician, 6 links, 5 joints
Joints:
- joint joint_2: origin xyz=-0.01175 0 0.114 rpy=1.570796325 -0.2 0 -> xyz=-0.01175 -0.01175 0.114 rpy=1.570796325 -0.2 0

Commit message: Fixed end effector angle by trigonometry in sim

File: src/magician-master/urdf/demo.urdf (robot description, URDF)
Before this commit: robot magician, 6 links, 5 joints
Joints:
- joint joint_7: origin xyz=-0.0328 0.02871 0 rpy=0 3.14159265 0 -> xyz=-0.0328 0.02871 0 rpy=0 3.14159265 -2.6
